File: hardware-2/DelSolClock/DelSolClock.kicad_sch (KiCad schematic)
At the start: 74 parts, among them J1 Conn_01x02_Male, J10 Conn_01x02_Male, J11 Conn_01x08_Male, J2 Conn_01x06, J3 Conn_01x02_Male, J4 Conn_01x02_Male, J5 Conn_01x02_Male, J6 CLOCK_BUTTONS, J7 Conn_01x02_Male, J8 Conn_01x02_Male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

Commit message: more progress on layout. Not done yet.
Parts:
- Y1: value DT-26 32.768KHz -> (none); footprint Crystal:Crystal_DS26_D2.0mm_L6.0mm_Horizontal_1EP_style1 -> (none)
Changed lines of the file:
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@@
     (in_bom yes) (on_board yes) (fields_autoplaced)
     (property "Reference" "Y1" (id 0) (at 86.36 99.0432 0))
-    (property "Value" "DT-26 32.768KHz" (id 1) (at 86.36 101.5801 0))
-    (property "Footprint" "Crystal:Crystal_DS26_D2.0mm_L6.0mm_Horizontal_1EP_style1" (id 2) (at 86.36 104.14 0)
+    (property "Value" "" (id 1) (at 86.36 101.5801 0))
+    (property "Footprint" "" (id 2) (at 86.36 104.14 0)
       (effects (font (size 1.27 1.27)) hide)
     )

Commit message: HW updates after testing the last prototype round. fixed PNP and NPN transistor pin mapping error (whoops) added keepouts and moved components inside of the board area. added holes for the rectangle LED footprints added a lot of silkscreen labels
Main remaining item is to adjust LED placement after testing.
Parts:
- Q1, Q2, Q3: value PZT2222A -> MMBT2222A; symbol Transistor_BJT:PZT2222A -> DelSolLib:MMBT2222A
- Y1: value (none) -> DT-26 32.768KHz; footprint (none) -> Crystal:Crystal_DS26_D2.0mm_L6.0mm_Horizontal_1EP_style1
Connections:
- net +12V: now also Q4.2 (E), Q5.2 (E), Q6.2 (E); no longer Q4.3 (C), Q5.3 (C), Q6.3 (C)
- net DTR: now also Q1.2 (E); no longer Q1.3 (E)
- net GND: now also Q3.2 (E); no longer Q3.3 (E)
- net GPIO0: now also Q1.3 (C); no longer Q1.2 (C)
- net RESET: now also Q2.3 (C); no longer Q2.2 (C)
- net RTS: now also Q2.2 (E); no longer Q2.3 (E)
- net input_divider5/IN: now also Q6.3 (C); no longer Q6.2 (E)
- net input_divider6/IN: now also Q5.3 (C); no longer Q5.2 (E)
- net input_divider7/IN: now also Q4.3 (C); no longer Q4.2 (E)
- net at BZ1.2 (+), D1.2 (A), TPBUZ1.1: now also Q3.3 (C); no longer Q3.2 (C)
Other:
- moved on the sheet: Q4, Q5, Q6
Changed lines of the file:
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@@
     (pin "2")
   )
-  (symbol (lib_id "Transistor_BJT:PZT2222A") (at 77.47 170.18 0) (unit 1)
+  (symbol (lib_id "DelSolLib:MMBT2222A") (at 77.47 170.18 0) (unit 1)
     (in_bom yes) (on_board yes) (fields_autoplaced)
     (property "Reference" "Q1" (id 0) (at 82.3214 169.3453 0)
       (effects (font (size 1.27 1.27)) (justify left))
     )
-    (property "Value" "PZT2222A" (id 1) (at 82.3214 171.8822 0)
+    (property "Value" "MMBT2222A" (id 1) (at 82.55 170.18 0)
       (effects (font (size 1.27 1.27)) (justify left))
     )
@@
       (effects (font (size 1.27 1.27) italic) (justify left) hide)
     )
-    (property "Datasheet" "https://www.onsemi.com/pub/Collateral/PN2222-D.PDF" (id 3) (at 77.47 170.18 0)
+    (property "Datasheet" "https://datasheet.lcsc.com/lcsc/1811081957_Jiangsu-Changjing-Electronics-Technology-Co---Ltd--MMBT2222A-1P_C8512.pdf" (id 3) (at 77.47 170.18 0)
       (effects (font (size 1.27 1.27)) (justify left) hide)
     )
@@
     (pin "2")
   )
-  (symbol (lib_id "Device:Q_PNP_BEC") (at 171.45 101.6 0) (mirror y) (unit 1)
-    (in_bom yes) (on_board yes) (fields_autoplaced)
-    (property "Reference" "Q5" (id 0) (at 166.5986 100.7653 0)
-      (effects (font (size 1.27 1.27)) (justify left))
-    )
-    (property "Value" "MMBT2907A" (id 1) (at 166.5986 103.3022 0)
-      (effects (font (size 1.27 1.27)) (justify left))
-    )
-    (property "Footprint" "Package_TO_SOT_SMD:SOT-23" (id 2) (at 166.37 99.06 0)
+  (symbol (lib_id "Device:Q_PNP_BEC") (at 171.45 101.6 180) (unit 1)
+    (in_bom yes) (on_board yes) (fields_autoplaced)
+    (property "Reference" "Q5" (id 0) (at 166.5987 100.7653 0)
+      (effects (font (size 1.27 1.27)) (justify left))
+    )
+    (property "Value" "MMBT2907A" (id 1) (at 166.5987 103.3022 0)
+      (effects (font (size 1.27 1.27)) (justify left))
+    )
+    (property "Footprint" "Package_TO_SOT_SMD:SOT-23" (id 2) (at 166.37 104.14 0)
       (effects (font (size 1.27 1.27)) hide)
     )
@@
     (pin "2")
   )
-  (symbol (lib_id "Device:Q_PNP_BEC") (at 138.43 101.6 0) (mirror y) (unit 1)
-    (in_bom yes) (on_board yes) (fields_autoplaced)
-    (property "Reference" "Q4" (id 0) (at 133.5786 100.7653 0)
-      (effects (font (size 1.27 1.27)) (justify left))
-    )
-    (property "Value" "MMBT2907A" (id 1) (at 133.5786 103.3022 0)
-      (effects (font (size 1.27 1.27)) (justify left))
-    )
-    (property "Footprint" "Package_TO_SOT_SMD:SOT-23" (id 2) (at 133.35 99.06 0)
+  (symbol (lib_id "Device:Q_PNP_BEC") (at 138.43 101.6 180) (unit 1)
+    (in_bom yes) (on_board yes) (fields_autoplaced)
+    (property "Reference" "Q4" (id 0) (at 133.5787 100.7653 0)
+      (effects (font (size 1.27 1.27)) (justify left))
+    )
+    (property "Value" "MMBT2907A" (id 1) (at 133.5787 103.3022 0)
+      (effects (font (size 1.27 1.27)) (justify left))
+    )
+    (property "Footprint" "Package_TO_SOT_SMD:SOT-23" (id 2) (at 133.35 104.14 0)
       (effects (font (size 1.27 1.27)) hide)
     )
@@
     (pin "2")
   )
-  (symbol (lib_id "Transistor_BJT:PZT2222A") (at 110.49 44.45 0) (unit 1)
+  (symbol (lib_id "DelSolLib:MMBT2222A") (at 110.49 44.45 0) (unit 1)
     (in_bom yes) (on_board yes) (fields_autoplaced)
     (property "Reference" "Q3" (id 0) (at 115.3414 43.6153 0)
       (effects (font (size 1.27 1.27)) (justify left))
     )
-    (property "Value" "PZT2222A" (id 1) (at 115.3414 46.1522 0)
+    (property "Value" "MMBT2222A" (id 1) (at 115.57 44.45 0)
       (effects (font (size 1.27 1.27)) (justify left))
     )
@@
       (effects (font (size 1.27 1.27) italic) (justify left) hide)
     )
-    (property "Datasheet" "https://www.onsemi.com/pub/Collateral/PN2222-D.PDF" (id 3) (at 110.49 44.45 0)
+    (property "Datasheet" "https://datasheet.lcsc.com/lcsc/1811081957_Jiangsu-Changjing-Electronics-Technology-Co---Ltd--MMBT2222A-1P_C8512.pdf" (id 3) (at 110.49 44.45 0)
       (effects (font (size 1.27 1.27)) (justify left) hide)
     )
@@
     (pin "2")
   )
-  (symbol (lib_id "Device:Q_PNP_BEC") (at 205.74 101.6 0) (mirror y) (unit 1)
-    (in_bom yes) (on_board yes) (fields_autoplaced)
-    (property "Reference" "Q6" (id 0) (at 200.8886 100.7653 0)
-      (effects (font (size 1.27 1.27)) (justify left))
-    )
-    (property "Value" "MMBT2907A" (id 1) (at 200.8886 103.3022 0)
-      (effects (font (size 1.27 1.27)) (justify left))
-    )
-    (property "Footprint" "Package_TO_SOT_SMD:SOT-23" (id 2) (at 200.66 99.06 0)
+  (symbol (lib_id "Device:Q_PNP_BEC") (at 205.74 101.6 180) (unit 1)
+    (in_bom yes) (on_board yes) (fields_autoplaced)
+    (property "Reference" "Q6" (id 0) (at 200.8887 100.7653 0)
+      (effects (font (size 1.27 1.27)) (justify left))
+    )
+    (property "Value" "MMBT2907A" (id 1) (at 200.8887 103.3022 0)
+      (effects (font (size 1.27 1.27)) (justify left))
+    )
+    (property "Footprint" "Package_TO_SOT_SMD:SOT-23" (id 2) (at 200.66 104.14 0)
       (effects (font (size 1.27 1.27)) hide)
     )
@@
     (in_bom yes) (on_board yes) (fields_autoplaced)
     (property "Reference" "Y1" (id 0) (at 86.36 99.0432 0))
-    (property "Value" "" (id 1) (at 86.36 101.5801 0))
-    (property "Footprint" "" (id 2) (at 86.36 104.14 0)
+    (property "Value" "DT-26 32.768KHz" (id 1) (at 86.36 101.5801 0))
+    (property "Footprint" "Crystal:Crystal_DS26_D2.0mm_L6.0mm_Horizontal_1EP_style1" (id 2) (at 86.36 104.14 0)
       (effects (font (size 1.27 1.27)) hide)
     )
@@
     (pin "1")
   )
-  (symbol (lib_id "Transistor_BJT:PZT2222A") (at 77.47 187.96 0) (mirror x) (unit 1)
+  (symbol (lib_id "DelSolLib:MMBT2222A") (at 77.47 187.96 0) (mirror x) (unit 1)
     (in_bom yes) (on_board yes) (fields_autoplaced)
     (property "Reference" "Q2" (id 0) (at 82.3214 187.1253 0)
       (effects (font (size 1.27 1.27)) (justify left))
     )
-    (property "Value" "PZT2222A" (id 1) (at 82.3214 189.6622 0)
+    (property "Value" "MMBT2222A" (id 1) (at 82.55 187.96 0)
       (effects (font (size 1.27 1.27)) (justify left))
     )
@@
       (effects (font (size 1.27 1.27) italic) (justify left) hide)
     )
-    (property "Datasheet" "https://www.onsemi.com/pub/Collateral/PN2222-D.PDF" (id 3) (at 77.47 187.96 0)
+    (property "Datasheet" "https://datasheet.lcsc.com/lcsc/1811081957_Jiangsu-Changjing-Electronics-Technology-Co---Ltd--MMBT2222A-1P_C8512.pdf" (id 3) (at 77.47 187.96 0)
       (effects (font (size 1.27 1.27)) (justify left) hide)
     )
@@
     )
     (path "/03a3adeb-e61a-4f7f-b2df-c747f3824a2d"
-      (reference "Q1") (unit 1) (value "PZT2222A") (footprint "Package_TO_SOT_SMD:SOT-23")
+      (reference "Q1") (unit 1) (value "MMBT2222A") (footprint "Package_TO_SOT_SMD:SOT-23")
     )
     (path "/e893f0dd-723f-4b52-b686-1067f2cb8778"
-      (reference "Q2") (unit 1) (value "PZT2222A") (footprint "Package_TO_SOT_SMD:SOT-23")
+      (reference "Q2") (unit 1) (value "MMBT2222A") (footprint "Package_TO_SOT_SMD:SOT-23")
     )
     (path "/82703eaf-ee57-455d-b591-d4f40ba10657"
-      (reference "Q3") (unit 1) (value "PZT2222A") (footprint "Package_TO_SOT_SMD:SOT-23")
+      (reference "Q3") (unit 1) (value "MMBT2222A") (footprint "Package_TO_SOT_SMD:SOT-23")
     )
     (path "/549e9541-43d0-4f23-aeaf-1c3e368d44f6"
