File: hardware/DelSolClock/DelSolClock.kicad_pcb (KiCad board)
At the start: 2 copper layers, 63.8 x 70.9 mm, 94 parts, among them J1 Conn_01x02_Male, J10 Conn_01x02_Male, J11 Conn_01x08_Male, J2 Conn_01x06, J3 Conn_01x02_Male, J4 Conn_01x02_Male, J5 Conn_01x02_Male, J6 CLOCK_BUTTONS, J7 Conn_01x02_Male, J8 Conn_01x02_Male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

Commit message: added missing 3V3 connection to the accelerometer CS pin, to select I2C mode.
Connections:
- C10 pad 1: Net-(C10-Pad1) -> Net-(J10-Pin_2)
- J10 pad 2: Net-(C10-Pad1) -> Net-(J10-Pin_2)
- R19 pad 2: Net-(C10-Pad1) -> Net-(J10-Pin_2)
- U6 pad 12: unconnected-(U6-Pad12) -> Net-(J10-Pin_2)
- U6 pad 5: Net-(C10-Pad1) -> Net-(J10-Pin_2)
- U6 pad 8: Net-(C10-Pad1) -> Net-(J10-Pin_2)
Routing:
- net Net-(J10-Pin_2): track 0.00 -> 20.8 mm
- net Net-(C10-Pad1): track 16.7 -> 0.00 mm
