File: hardware/DelSolClock/DelSolClock.kicad_sch (KiCad schematic)
At the start: 74 parts, among them J1 Conn_01x02_Male, J10 Conn_01x02_Male, J11 Conn_01x08_Male, J2 Conn_01x06, J3 Conn_01x02_Male, J4 Conn_01x02_Male, J5 Conn_01x02_Male, J6 CLOCK_BUTTONS, J7 Conn_01x02_Male, J8 Conn_01x02_Male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

Commit message: added missing 3V3 connection to the accelerometer CS pin, to select I2C mode.
Connections:
- net at C10.1, J10.2 (Pin_2), R19.2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: now also U6.12 (CS)
- no-connect marks 22 -> 21
Changed lines of the file:
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@@
+	)
+	(junction
+		(at 241.3 45.72)
+		(diameter 0)
+		(color 0 0 0 0)
 	)
 	(junction
@@
 	)
 	(no_connect
-		(at 226.06 69.85)
-	)
-	(no_connect
 		(at 226.06 59.69)
 	)
@@
 	(wire
 		(pts
+			(xy 226.06 69.85) (xy 213.36 69.85)
+		)
+		(stroke
+			(width 0)
+			(type default)
+		)
+	)
+	(wire
+		(pts
 			(xy 60.96 177.8) (xy 60.96 187.96)
 		)
@@
 	(wire
 		(pts
+			(xy 241.3 45.72) (xy 241.3 46.99)
+		)
+		(stroke
+			(width 0)
+			(type default)
+		)
+	)
+	(wire
+		(pts
 			(xy 16.51 45.72) (xy 27.94 45.72)
 		)
@@
 	(wire
 		(pts
+			(xy 213.36 69.85) (xy 213.36 45.72)
+		)
+		(stroke
+			(width 0)
+			(type default)
+		)
+	)
+	(wire
+		(pts
 			(xy 190.5 154.94) (xy 195.58 154.94)
 		)
@@
 	(wire
 		(pts
+			(xy 213.36 45.72) (xy 241.3 45.72)
+		)
+		(stroke
+			(width 0)
+			(type default)
+		)
+	)
+	(wire
+		(pts
 			(xy 80.01 162.56) (xy 82.55 162.56)
 		)
@@
 	(wire
 		(pts
-			(xy 241.3 33.02) (xy 241.3 46.99)
-		)
-		(stroke
+			(xy 241.3 33.02) (xy 241.3 45.72)
+		)
+		(stroke
